File: GPSClockISA.brd (EAGLE design)
At the start: 98.7 x 99 mm, 37 parts, among them IC2 27C512AP, IC3 8250/16450, IC6 74HC138N, IC7 74HC138N, IC8 74HC688N, IC9 74LS85N, X1 53047-08, X2 1.8432MHz

Commit message: Add files via upload
Parts:
- added JP4, JP5, JP6: (no value), pinhead-2:1X03
- moved IC9 4.02 mm to (12.7, 53.3), turned to 0 degrees
- moved C5 4.02 mm to (25.4, 69.8)
- moved IC8 3.59 mm to (35.6, 52.1)
- moved C8 2.84 mm to (50.8, 73.7)
- moved C7 2.84 mm to (66.7, 61.0)
- moved IC6 2.84 mm to (57.1, 47.0)
- moved RN1 2.54 mm to (25.4, 78.7)
- moved S3 2.54 mm to (16.5, 69.8)
- moved S2 2.54 mm to (34.3, 71.1)
- moved R1 1.80 mm to (70.5, 64.8)
- moved LED1 1.27 mm to (97.8, 64.8)
- moved LED2 1.27 mm to (96.5, 64.8)
- moved D2 1.27 mm to (57.8, 61.6)
- moved IC3 1.27 mm to (82.5, 36.8)
- moved JMP1 1.27 mm to (67.3, 67.3)
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Connections:
- new net N$16: IC2.27, JP4.2
- new net N$19: IC2.1, JP5.2
- new net N$22: IC2.24, JP6.2
- net +5V: now also JP6.1
- net BA14: now also JP4.3, JP5.3; no longer IC2.27
- net BA15: now also JP5.1; no longer IC2.1
- net BA9: now also JP6.3; no longer IC2.24
- net GND: now also IC3.25
- net MEMW: now also JP4.1
- net RI: now also IC3.39
Routing:
- net MEMW: track 0.00 -> 119.8 mm, vias 0 -> 6
- net BD6: track 114.9 -> 217.8 mm, vias 2 -> 5
- net VCC: track 53.0 -> 127.5 mm, vias 0 -> 3
- net IRQ3: track 114.2 -> 184.6 mm, vias 6 -> 4
- net MEMR: track 58.6 -> 125.4 mm, vias 5 -> 7
- net RI: track 0.00 -> 65.8 mm, vias 0 -> 2
- net BD0: track 73.2 -> 130.8 mm, vias 3 -> 7
- net IRQ4: track 172.2 -> 114.6 mm, vias 2 -> 3
- net BA15: track 184.0 -> 137.6 mm, vias 5 -> 6
- net BA8: track 96.5 -> 70.6 mm, vias 4 -> 3
- net BA12: track 104.0 -> 129.6 mm
- net BD5: track 125.8 -> 102.1 mm, vias 4 -> 8
- net BA14: track 106.0 -> 124.3 mm, vias 3 -> 6
- net BD1: track 96.3 -> 114.1 mm, vias 5 -> 3
- net BA6: track 76.4 -> 59.0 mm
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Other:
- board size 98.7 x 99 mm -> 98.7 x 86.3 mm
- board text added: "GPSClockISA (C) Dario's Automation 2025"
