File: GPSClockISA.sch (EAGLE design)
At the start: 37 parts, among them IC2 27C512AP, IC3 8250/16450, IC6 74HC138N, IC7 74HC138N, IC8 74HC688N, IC9 74LS85N, X1 53047-08, X2 1.8432MHz

Commit message: Add files via upload
Parts:
- added JP4, JP5, JP6: (no value), pinhead-2:PINHD-1X03_2.54
Connections:
- new net N$16: IC2.A14, JP4.2
- new net N$19: IC2.A15, JP5.2
- new net N$22: IC2.A9, JP6.2
- net +5V: now also JP6.1
- net BA14: now also JP4.3, JP5.3; no longer IC2.A14
- net BA15: now also JP5.1; no longer IC2.A15
- net BA9: now also JP6.3; no longer IC2.A9
- net GND: now also IC3.ADS
- net MEMW: now also JP4.1
- net RI: now also IC3.RI
Other:
- note added: "anche 27256, 2864, 28128 ecc"
- moved on the sheet: IC2
