File: GPSClockISA.sch (EAGLE design)
At the start: 45 parts, among them IC1 74LS85N, IC2 74HC138N, IC3 27C512AP, IC4 74HC688N, IC5 8250/16450, IC6 74HC138N, X1 1.8432MHz, X2 53047-08

Commit message: Add files via upload
Parts:
- added H1, H2: MOUNT-HOLEM3, holes:MOUNT-HOLEM3
- added JP10, JP7, JP8, JP9: (no value), pinhead:PINHD-1X1
Connections:
- new net N$26: IC5.DSR, JP7.1
- new net N$27: IC5.CTS, JP8.1
- new net N$28: IC5.DTR, JP9.1
- new net N$29: IC5.RTS, JP10.1
- net BA13: now also JMP1-0R.1
- net BA15: no longer JMP1-0R.1
Changed lines of the file:
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@@
 <part name="JMP2" library="jump-0r-smd" deviceset="0R-JUMP" device="C"/>
 <part name="JMP1" library="jump-0r-smd" deviceset="0R-JUMP" device="C"/>
+<part name="JP7" library="pinhead" deviceset="PINHD-1X1" device=""/>
+<part name="JP8" library="pinhead" deviceset="PINHD-1X1" device=""/>
+<part name="JP9" library="pinhead" deviceset="PINHD-1X1" device=""/>
+<part name="JP10" library="pinhead" deviceset="PINHD-1X1" device=""/>
+<part name="H1" library="holes" deviceset="MOUNT-HOLE" device="M3"/>
+<part name="H2" library="holes" deviceset="MOUNT-HOLE" device="M3"/>
 </parts>
 <sheets>
@@
 <instance part="JMP1" gate="-0R" x="91.44" y="157.48"/>
 <instance part="JMP1" gate="G$2" x="88.9" y="160.02"/>
+<instance part="JP7" gate="G$1" x="251.46" y="121.92"/>
+<instance part="JP8" gate="G$1" x="251.46" y="116.84"/>
+<instance part="JP9" gate="G$1" x="251.46" y="111.76"/>
+<instance part="JP10" gate="G$1" x="251.46" y="106.68"/>
+<instance part="H1" gate="G$1" x="48.26" y="200.66"/>
+<instance part="H2" gate="G$1" x="68.58" y="200.66"/>
 </instances>
 <busses>
@@
 <label x="172.72" y="180.34" size="1.778" layer="95"/>
 </segment>
+<segment>
+<pinref part="JMP1" gate="-0R" pin="1"/>
+<wire x1="91.44" y1="160.02" x2="76.2" y2="160.02" width="0.1524" layer="91"/>
+<label x="78.74" y="160.02" size="1.778" layer="95"/>
+</segment>
 </net>
 <net name="BA14" class="0">
@@
 <wire x1="91.44" y1="45.72" x2="91.44" y2="55.88" width="0.1524" layer="91"/>
 <label x="91.44" y="50.8" size="1.778" layer="95" rot="R90"/>
-</segment>
-<segment>
-<pinref part="JMP1" gate="-0R" pin="1"/>
-<wire x1="91.44" y1="160.02" x2="76.2" y2="160.02" width="0.1524" layer="91"/>
-<label x="78.74" y="160.02" size="1.778" layer="95"/>
 </segment>
 </net>
@@
 </segment>
 </net>
+<net name="N$26" class="0">
+<segment>
+<pinref part="IC5" gate="G$1" pin="DSR"/>
+<wire x1="220.98" y1="114.3" x2="238.76" y2="114.3" width="0.1524" layer="91"/>
+<wire x1="238.76" y1="114.3" x2="238.76" y2="121.92" width="0.1524" layer="91"/>
+<pinref part="JP7" gate="G$1" pin="1"/>
+<wire x1="238.76" y1="121.92" x2="248.92" y2="121.92" width="0.1524" layer="91"/>
+</segment>
+</net>
+<net name="N$27" class="0">
+<segment>
+<pinref part="IC5" gate="G$1" pin="CTS"/>
+<wire x1="220.98" y1="111.76" x2="241.3" y2="111.76" width="0.1524" layer="91"/>
+<wire x1="241.3" y1="111.76" x2="241.3" y2="116.84" width="0.1524" layer="91"/>
+<pinref part="JP8" gate="G$1" pin="1"/>
+<wire x1="241.3" y1="116.84" x2="248.92" y2="116.84" width="0.1524" layer="91"/>
+</segment>
+</net>
+<net name="N$28" class="0">
+<segment>
+<pinref part="IC5" gate="G$1" pin="DTR"/>
+<wire x1="220.98" y1="109.22" x2="243.84" y2="109.22" width="0.1524" layer="91"/>
+<wire x1="243.84" y1="109.22" x2="243.84" y2="111.76" width="0.1524" layer="91"/>
+<pinref part="JP9" gate="G$1" pin="1"/>
+<wire x1="243.84" y1="111.76" x2="248.92" y2="111.76" width="0.1524" layer="91"/>
+</segment>
+</net>
+<net name="N$29" class="0">
+<segment>
+<pinref part="IC5" gate="G$1" pin="RTS"/>
+<pinref part="JP10" gate="G$1" pin="1"/>
+<wire x1="220.98" y1="106.68" x2="248.92" y2="106.68" width="0.1524" layer="91"/>
+</segment>
+</net>
