File: GPSClockISAsmd.brd (EAGLE design)
At the start: 98.7 x 83.8 mm, 45 parts, among them IC1 74LS85N, IC2 74HC138N, IC3 27C512AP, IC4 74HC688N, IC5 8250/16450, IC6 74HC138N, X1 1.8432MHz, X2 53047-08

Commit message: Add files via upload
Parts:
- IC1: value 74LS85N -> 74LS85D; device 74xx-eu:DIL16 -> 74xx-eu:SO16
- IC2, IC6: value 74HC138N -> 74LS138D; device 74xx-eu:DIL16 -> 74xx-eu:SO16
- IC4: value 74HC688N -> 74LS688DW; device 74xx-eu:DIL20 -> 74xx-eu:SO20W
- IC5: value 8250/16450 -> (none); device micro-intel:DIL40 -> micro-intel:PLCC44
- moved C9 39.4 mm to (96.5, 14.0), turned to 0 degrees
- moved X1 26.7 mm to (96.5, 20.3)
- moved JP1 26.4 mm to (59.1, 15.2), turned to 0 degrees
- moved IC2 26.2 mm to (83.8, 39.4), turned to 0 degrees
- moved JP4 20.1 mm to (40.6, 29.8)
- moved R1 15.2 mm to (70.5, 49.5)
- moved D1 14.0 mm to (57.8, 46.4)
- moved C8 14.0 mm to (96.5, 26.7)
- moved JMP3 14.0 mm to (67.3, 53.3)
- moved C10 12.7 mm to (50.8, 59.7)
- moved C7 12.7 mm to (66.7, 48.3)
- moved JP3 12.7 mm to (66.7, 61.0)
- moved LED1 12.7 mm to (97.8, 44.5)
- moved LED2 12.7 mm to (96.5, 44.5)
- moved X2 12.7 mm to (73.0, 64.1)
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Connections:
- net +5V: now also IC5.14, IC5.15, IC5.21, IC5.25, IC5.44; no longer IC5.12, IC5.13, IC5.19, IC5.22, IC5.40
- net BA0: now also IC5.31; no longer IC5.28
- net BA1: now also IC5.30; no longer IC5.27
- net BA2: now also IC5.29; no longer IC5.26
- net BD0: now also IC5.2; no longer IC5.1
- net BD1: now also IC5.3; no longer IC5.2
- net BD2: now also IC5.4; no longer IC5.3
- net BD3: now also IC5.5; no longer IC5.4
- net BD4: now also IC5.6; no longer IC5.5
- net BD5: now also IC5.7; no longer IC5.6
- net BD6: now also IC5.8; no longer IC5.7
- net BD7: now also IC5.9; no longer IC5.8
- net GND: now also IC5.22, IC5.28; no longer IC5.20, IC5.25
- net IOR: now also IC5.24; no longer IC5.21
- net IOW: now also IC5.20; no longer IC5.18
- net N$14: now also IC5.10, IC5.17; no longer IC5.15, IC5.9
- net N$15: now also IC5.19; no longer IC5.17
- net N$17: now also IC5.18; no longer IC5.16
- net N$25: now also IC5.16; no longer IC5.14
- net N$7: now also IC5.33; no longer IC5.30
- net OUT1: now also IC5.38; no longer IC5.34
- net OUT2: now also IC5.35; no longer IC5.31
- net RESET: now also IC5.39; no longer IC5.35
- net RI: now also IC5.43; no longer IC5.39
- net RX: now also IC5.13; no longer IC5.11
- net TX: now also IC5.11; no longer IC5.10
Other:
- board size 98.7 x 83.8 mm -> 98.7 x 71.1 mm
