File: GPSClockISAsmd.sch (EAGLE design)
At the start: 45 parts, among them IC1 74LS85N, IC2 74HC138N, IC3 27C512AP, IC4 74HC688N, IC5 8250/16450, IC6 74HC138N, X1 1.8432MHz, X2 53047-08

Commit message: Add files via upload
Parts:
- IC1: value 74LS85N -> 74LS85D; device 74xx-eu:74LS85N -> 74xx-eu:74LS85D
- IC2, IC6: value 74HC138N -> 74LS138D; device 74xx-eu:74HC138N -> 74xx-eu:74LS138D
- IC4: value 74HC688N -> 74LS688DW; device 74xx-eu:74HC688N -> 74xx-eu:74LS688DW
- IC5: value 8250/16450 -> (none); device micro-intel:8250 -> micro-intel:8250PLCC
