File: GPSClock.brd (EAGLE design)
At the start: 39 x 52.1 mm, 23 parts, among them IC1 78M03, IC2 MAX202CPESOIC, M1 2.1MMJACKTHM, X1 53047-08

Commit message: Add files via upload
Parts:
- added F2, F3: FIDUCIAL, adafruit:FIDUCIAL_1MM
- moved M1 11.6 mm to (4.45, 0.00), turned to 180 degrees
Routing:
- net +24V: track 6.76 -> 39.0 mm, vias 0 -> 2
- net GND: track 140.6 -> 157.3 mm
Other:
- board text added: "12V"
- board text added: "RS232 / 1Hz"
Changed lines of the file:
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@@
 <?xml version="1.0" encoding="utf-8"?>
 <!DOCTYPE eagle SYSTEM "eagle.dtd">
-<eagle version="7.7.0">
+<eagle version="7.2.0">
 <drawing>
 <settings>
@@
 <text x="38.1" y="50.8" size="1.4224" layer="16" rot="MR270">GPSClock
 Dario's Automation 2025</text>
-<rectangle x1="0" y1="0" x2="2.54" y2="20.32" layer="16"/>
-<rectangle x1="2.54" y1="6.35" x2="15.24" y2="19.05" layer="16"/>
 <rectangle x1="29.21" y1="0" x2="39.37" y2="12.7" layer="16"/>
 <rectangle x1="34.29" y1="12.7" x2="39.37" y2="20.32" layer="16"/>
@@
 <rectangle x1="20.32" y1="33.02" x2="24.13" y2="35.56" layer="16"/>
 <rectangle x1="22.86" y1="31.75" x2="24.13" y2="33.02" layer="16"/>
+<text x="17.78" y="49.53" size="1.778" layer="1">RS232 / 1Hz</text>
+<text x="6.35" y="12.7" size="1.778" layer="1">12V</text>
+<rectangle x1="2.54" y1="0" x2="11.43" y2="2.54" layer="16"/>
+<rectangle x1="2.54" y1="2.54" x2="5.08" y2="6.35" layer="16"/>
+<rectangle x1="0" y1="0" x2="2.54" y2="6.35" layer="16"/>
+<rectangle x1="0" y1="6.35" x2="1.27" y2="20.32" layer="16"/>
+<rectangle x1="1.27" y1="13.97" x2="13.97" y2="15.24" layer="16"/>
+<rectangle x1="8.89" y1="7.62" x2="13.97" y2="13.97" layer="16"/>
 </plain>
 <attributes>
@@
 <element name="LED1" library="led" package="CHIPLED_0805" value="verde" x="1.905" y="21.59" rot="R90"/>
 <element name="LED2" library="adafruit" package="LED3MM" value="verde" x="2.3" y="22.86" rot="R180"/>
-<element name="M1" library="adafruit" package="PJ-102A" value="2.1MMJACKTHM" x="6.35" y="11.43"/>
+<element name="M1" library="adafruit" package="PJ-102A" value="2.1MMJACKTHM" x="4.445" y="0" rot="R180"/>
 <element name="R1" library="resistor" package="R0805" value="470" x="19.685" y="20.955" rot="R90"/>
 <element name="X1" library="con-molex" package="53047-08" value="53047-08" x="33.02" y="24.13">
@@
 <element name="C9" library="resistor" package="SMC_C" value="10u" x="10.16" y="30.48" rot="R180"/>
 <element name="D3" library="diode" package="SMB" value="ES2D" x="13.335" y="20.32" rot="R180"/>
+<element name="F3" library="adafruit" package="FIDUCIAL_1MM" value="FIDUCIAL" x="1.27" y="12.7"/>
+<element name="F2" library="adafruit" package="FIDUCIAL_1MM" value="FIDUCIAL" x="38.1" y="50.8"/>
 </elements>
 <signals>
@@
 <wire x1="33.7185" y1="24.5745" x2="33.645" y2="24.58" width="0.508" layer="1"/>
 <wire x1="24.2316" y1="22.0599" x2="24.2316" y2="21.6027" width="0.508" layer="16"/>
-<wire x1="28.2321" y1="26.0604" x2="24.2316" y2="22.0599" width="0.508" layer="16"/>
+<wire x1="28.2321" y1="26.0604" x2="25.88895" y2="23.71725" width="0.508" layer="16"/>
+<wire x1="25.88895" y1="23.71725" x2="24.2316" y2="22.0599" width="0.508" layer="16"/>
 <wire x1="32.8041" y1="26.0604" x2="28.2321" y2="26.0604" width="0.508" layer="16"/>
 <wire x1="33.6042" y1="25.2603" x2="32.8041" y2="26.0604" width="0.508" layer="16"/>
@@
 <wire x1="37.6047" y1="20.1168" x2="37.78" y2="20.32" width="0.508" layer="1"/>
 <wire x1="34.29" y1="10.1727" x2="34.29" y2="10.16" width="0.508" layer="1"/>
-<wire x1="7.4295" y1="9.0297" x2="15.2019" y2="9.0297" width="0.508" layer="1"/>
-<wire x1="6.5151" y1="8.1153" x2="7.4295" y2="9.0297" width="0.508" layer="1"/>
-<wire x1="15.2019" y1="9.0297" x2="15.24" y2="9.05" width="0.508" layer="1"/>
-<wire x1="6.5151" y1="8.1153" x2="6.45" y2="8.04" width="0.508" layer="1"/>
-<wire x1="3.5433" y1="5.1435" x2="1.8288" y2="5.1435" width="0.508" layer="1"/>
-<wire x1="6.2865" y1="7.8867" x2="3.5433" y2="5.1435" width="0.508" layer="1"/>
-<wire x1="1.8288" y1="5.1435" x2="1.75" y2="5.14" width="0.508" layer="1"/>
-<wire x1="6.2865" y1="7.8867" x2="6.45" y2="8.04" width="0.508" layer="1"/>
 <wire x1="24.1173" y1="20.3454" x2="24.1173" y2="21.4884" width="0.508" layer="1"/>
 <wire x1="18.8595" y1="15.0876" x2="24.1173" y2="20.3454" width="0.508" layer="1"/>
@@
 <wire x1="24.1173" y1="21.4884" x2="24.13" y2="21.59" width="0.508" layer="1"/>
 <wire x1="15.3162" y1="9.2583" x2="15.24" y2="9.05" width="0.508" layer="1"/>
-<wire x1="1.4859" y1="15.0876" x2="1.4859" y2="17.6022" width="0.508" layer="1"/>
-<wire x1="7.3152" y1="9.2583" x2="1.4859" y2="15.0876" width="0.508" layer="1"/>
 <wire x1="1.4859" y1="17.6022" x2="1.295" y2="17.78" width="0.508" layer="1"/>
-<wire x1="7.3152" y1="9.2583" x2="6.45" y2="8.04" width="0.508" layer="1"/>
+<wire x1="6.1722" y1="3.429" x2="4.4577" y2="3.429" width="0.6096" layer="1"/>
+<wire x1="9.0297" y1="6.2865" x2="6.1722" y2="3.429" width="0.6096" layer="1"/>
+<wire x1="4.4577" y1="3.429" x2="4.345" y2="3.39" width="0.508" layer="1"/>
+<wire x1="9.0297" y1="6.2865" x2="9.045" y2="6.29" width="0.508" layer="1"/>
+<wire x1="12.3444" y1="6.4008" x2="9.2583" y2="6.4008" width="0.6096" layer="1"/>
+<wire x1="13.8303" y1="7.8867" x2="12.3444" y2="6.4008" width="0.508" layer="1"/>
+<wire x1="14.6304" y1="7.8867" x2="13.8303" y2="7.8867" width="0.508" layer="1"/>
+<wire x1="15.2019" y1="8.4582" x2="14.6304" y2="7.8867" width="0.508" layer="1"/>
+<wire x1="15.2019" y1="8.8011" x2="15.2019" y2="8.4582" width="0.508" layer="1"/>
+<wire x1="9.2583" y1="6.4008" x2="9.045" y2="6.29" width="0.508" layer="1"/>
+<wire x1="15.2019" y1="8.8011" x2="15.24" y2="9.05" width="0.508" layer="1"/>
+<wire x1="11.43" y1="38.1762" x2="25.88895" y2="23.71725" width="0.508" layer="16"/>
+<wire x1="11.43" y1="48.26" x2="11.43" y2="38.1762" width="0.508" layer="16"/>
 <wire x1="0.855" y1="21.59" x2="1.03" y2="22.86" width="0" layer="19" extent="1-1"/>
 <wire x1="1.3716" y1="17.8308" x2="0.855" y2="21.59" width="0" layer="19" extent="1-1"/>
@@
 <contactref element="M1" pad="TIP"/>
 <contactref element="D1" pad="A"/>
-<wire x1="6.858" y1="2.5146" x2="13.0302" y2="2.5146" width="0.508" layer="1"/>
-<wire x1="6.5151" y1="2.1717" x2="6.858" y2="2.5146" width="0.508" layer="1"/>
 <wire x1="13.0302" y1="2.5146" x2="13.04" y2="2.54" width="0.508" layer="1"/>
-<wire x1="6.5151" y1="2.1717" x2="6.45" y2="2.14" width="0.508" layer="1"/>
+<wire x1="15.5448" y1="5.1435" x2="13.1445" y2="2.7432" width="0.508" layer="1"/>
+<wire x1="15.5448" y1="5.9436" x2="15.5448" y2="5.1435" width="0.508" layer="16"/>
+<wire x1="15.7734" y1="6.1722" x2="15.5448" y2="5.9436" width="0.508" layer="16"/>
+<wire x1="15.7734" y1="19.2024" x2="15.7734" y2="6.1722" width="0.508" layer="16"/>
+<wire x1="15.2019" y1="19.7739" x2="15.7734" y2="19.2024" width="0.508" layer="16"/>
+<wire x1="5.9436" y1="19.7739" x2="15.2019" y2="19.7739" width="0.508" layer="16"/>
+<wire x1="5.9436" y1="19.431" x2="5.9436" y2="19.7739" width="0.508" layer="1"/>
+<wire x1="4.4577" y1="17.9451" x2="5.9436" y2="19.431" width="0.508" layer="1"/>
+<wire x1="4.4577" y1="9.3726" x2="4.4577" y2="17.9451" width="0.508" layer="1"/>
+<wire x1="13.1445" y1="2.7432" x2="13.04" y2="2.54" width="0.508" layer="1"/>
+<wire x1="4.4577" y1="9.3726" x2="4.345" y2="9.29" width="0.508" layer="1"/>
+<via x="15.5448" y="5.1435" extent="1-16" drill="0.6096"/>
+<via x="5.9436" y="19.7739" extent="1-16" drill="0.6096"/>
 </signal>
 <signal name="CTS">
