File: GPSClock.sch (EAGLE design)
At the start: 23 parts, among them IC1 78M03, IC2 MAX202CPESOIC, M1 2.1MMJACKTHM, X1 53047-08

Commit message: Add files via upload
Parts:
- added F2, F3: FIDUCIAL, adafruit:FIDUCIAL
Other:
- note added: "il regolatore non dovrebbe servire Neo modulo ha regolatore on board"
Changed lines of the file:
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@@
 <part name="C9" library="resistor" deviceset="CPOL-EU" device="SMCC" value="10u"/>
 <part name="D3" library="diode" deviceset="ES2D" device=""/>
+<part name="F3" library="adafruit" deviceset="FIDUCIAL" device=""/>
+<part name="F2" library="adafruit" deviceset="FIDUCIAL" device=""/>
 </parts>
 <sheets>
@@
 <text x="180.34" y="35.56" size="1.778" layer="91">occhio: questo e 1.25 ma dovrebbe andare lo stesso</text>
 <text x="177.8" y="2.54" size="1.778" layer="91">Fasttrax</text>
+<text x="40.64" y="43.18" size="1.778" layer="91">il regolatore non dovrebbe servire
+Neo modulo ha regolatore on board</text>
 </plain>
 <instances>
@@
 <instance part="C9" gate="G$1" x="101.6" y="22.86"/>
 <instance part="D3" gate="G$1" x="58.42" y="27.94" rot="R90"/>
+<instance part="F3" gate="G$1" x="8.89" y="93.98" rot="R90"/>
+<instance part="F2" gate="G$1" x="8.89" y="81.28" rot="R90"/>
 </instances>
 <busses>
@@
 </schematic>
 </drawing>
+<compatibility>
+<note version="6.3" minversion="6.2.2" severity="warning">
+Since Version 6.2.2 text objects can contain more than one line,
+which will not be processed correctly with this version.
+</note>
+</compatibility>
 </eagle>
